File: board/mididude/mididude.kicad_sch (KiCad schematic)
At the start: 26 parts, among them J1 Conn_01x03_Pin, J10 Conn_01x03_Pin, J2 Conn_01x03_Pin, J3 Conn_01x03_Pin, J4 Conn_01x03_Pin, J5 Conn_01x03_Pin, J6 Conn_01x03_Pin, J7 Conn_01x03_Pin, J8 Conn_01x03_Pin, J9 Conn_01x03_Pin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

Commit message: Pretty good firmware
Parts:
- R9: value 20 -> 100
Changed lines of the file:
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@@
 			)
 		)
-		(property "Value" "20"
+		(property "Value" "100"
 			(at 190.5 67.3099 0)
 			(effects
